Commit message: added gazebo control

File: description/robot.urdf.xacro (robot description, xacro)
@@ -2,3 +2,4 @@
 <robot xmlns:xacro="http://www.ros.org/wiki/xacro"  name="robot">
    <xacro:include filename="robot_core.xacro"/>
+   <xacro:include filename="gazebo_control.xacro"/>
 </robot>

File: description/robot_core.xacro (robot description, xacro)
@@ -41,4 +41,7 @@
     </xacro:inertial_box>
   </link>
+  <gazebo reference="chassis">
+    <material>Gazebo/White</material>
+  </gazebo>
   <!-- LEFT WHEEL LINK -->
   <joint name="left_wheel_joint" type="continuous">
@@ -64,4 +67,7 @@
     </xacro:inertial_cylinder>
   </link>
+  <gazebo reference="left_wheel">
+    <material>Gazebo/Blue</material>
+  </gazebo>
     <!-- RIGHT WHEEL LINK -->
   <joint name="right_wheel_joint" type="continuous">
@@ -87,4 +93,7 @@
     </xacro:inertial_cylinder>
   </link>
+  <gazebo reference="right_wheel">
+    <material>Gazebo/Blue</material>
+  </gazebo>
   <!-- CASTER WHEEL LINK -->
   <joint name="caster_wheel_joint" type="fixed">
@@ -109,3 +118,8 @@
     </xacro:inertial_sphere>
   </link>
+  <gazebo reference="caster_wheel">
+    <material>Gazebo/Black</material>
+    <mu1 value="0.001"/>
+    <mu2 value="0.001"/>
+  </gazebo>
 </robot>

Commit message: added lidar

File: description/robot.urdf.xacro (robot description, xacro)
@@ -3,3 +3,4 @@
    <xacro:include filename="robot_core.xacro"/>
    <xacro:include filename="gazebo_control.xacro"/>
+   <xacro:include filename="lidar.xacro"/>
 </robot>

File: description/robot_core.xacro (robot description, xacro)
@@ -13,4 +13,7 @@
   <material name="black">
     <color rgba="0 0 0 1"/>
+  </material>
+   <material name="red">
+    <color rgba="1 0 0 1"/>
   </material>
   <!-- BASE LINK -->

Commit message: fixed gazebo issues

File: description/robot.urdf.xacro (robot description, xacro)
@@ -1,7 +1,12 @@
 <?xml version="1.0"?>
 <robot xmlns:xacro="http://www.ros.org/wiki/xacro"  name="robot">
+   <xacro:arg name="use_ros2_control" default="true"/>
+   <xacro:if value="$(arg use_ros2_control)">
+         <xacro:include filename="ros2_control.xacro"/>
+   </xacro:if>
+   <xacro:unless value="$(arg use_ros2_control)">
+         <xacro:include filename="gazebo_control.xacro"/>
+   </xacro:unless>
    <xacro:include filename="robot_core.xacro"/>
-   <!-- <xacro:include filename="gazebo_control.xacro"/> -->
-   <xacro:include filename="ros2_control.xacro"/>
    <xacro:include filename="lidar.xacro"/>
    <xacro:include filename="camera.xacro"/>

File: description/robot_core.xacro (robot description, xacro)
@@ -63,5 +63,5 @@
     <collision>
         <geometry>
-            <cylinder radius="0.05" length="0.04"/>
+            <sphere radius="0.05"/>
         </geometry>
     </collision>
@@ -89,5 +89,5 @@
     <collision>
         <geometry>
-            <cylinder radius="0.05" length="0.04"/>
+            <sphere radius="0.05"/>
         </geometry>
     </collision>
